File: hardware/control_board/control_board.kicad_pcb (KiCad board)
At the start: 2 copper layers, 101.6 x 53.3 mm, 13 parts, among them P1 Digital, P10 CONN_01X01, P11 CONN_01X01, P12 CONN_01X01, P13 CONN_01X01, P2 Power, P3 Analog, P4 Analog, P5 PWM, P6 PWM, P7 Communication, P8 CONN_01X01, P9 CONN_01X01

Commit message: control board schematic
Parts:
- removed P10, P11, P12, P13, P8, P9: CONN_01X01, Socket_Arduino_Mega:Arduino_1pin
- added A1: Pololu_Breakout_A4988, Module:Pololu_Breakout-16_15.2x20.3mm, F.Cu at (169.5, 89.5)
- added A2: Pololu_Breakout_A4988, Module:Pololu_Breakout-16_15.2x20.3mm, F.Cu at (169.5, 113.0)
- added A3: Pololu_Breakout_A4988, Module:Pololu_Breakout-16_15.2x20.3mm, F.Cu at (131.4, 113.0)
- added A4: Pololu_Breakout_A4988, Module:Pololu_Breakout-16_15.2x20.3mm, F.Cu at (131.4, 89.5)
- added C1: 100uF, Capacitor_THT:CP_Radial_D12.5mm_P5.00mm, F.Cu at (106.0, 200.8)
- added C2: 100uF, Capacitor_THT:CP_Radial_D12.5mm_P5.00mm, F.Cu at (106.0, 214.9)
- added C3: 100uF, Capacitor_THT:CP_Radial_D12.5mm_P5.00mm, F.Cu at (120.4, 200.8)
- added C4: 100uF, Capacitor_THT:CP_Radial_D12.5mm_P5.00mm, F.Cu at (120.4, 214.9)
- added J1: PWR_SWITCHES, TerminalBlock_4Ucon:TerminalBlock_4Ucon_1x04_P3.50mm_Horizontal, F.Cu at (114.9, 139.7)
- added J10: MO2_SW_FW, Connector_Molex:Molex_Nano-Fit_105309-xx03_1x03_P2.50mm_Vertical, F.Cu at (148.6, 168.3)
- added J11: MO3_SW_FW, Connector_Molex:Molex_Nano-Fit_105309-xx03_1x03_P2.50mm_Vertical, F.Cu at (140.2, 178.8)
- added J12: MO0_SW_BW, Connector_Molex:Molex_Nano-Fit_105309-xx03_1x03_P2.50mm_Vertical, F.Cu at (160.4, 163.1)
- added J13: MO1_SW_BW, Connector_Molex:Molex_Nano-Fit_105309-xx03_1x03_P2.50mm_Vertical, F.Cu at (148.6, 178.8)
- added J14: MO2_SW_BW, Connector_Molex:Molex_Nano-Fit_105309-xx03_1x03_P2.50mm_Vertical, F.Cu at (177.1, 155.5)
- added J15: MO3_SW_BW, Connector_Molex:Molex_Nano-Fit_105309-xx03_1x03_P2.50mm_Vertical, F.Cu at (157.0, 173.6)
- added J2: UI_SWITCHES, TerminalBlock_4Ucon:TerminalBlock_4Ucon_1x04_P3.50mm_Horizontal, F.Cu at (157.9, 146.7)
- added J3: ATX-24, Connector_Molex:Molex_Mini-Fit_Jr_5569-24A2_2x12_P4.20mm_Horizontal, F.Cu at (108.0, 118.1)
- added J4: MOT0, TerminalBlock_4Ucon:TerminalBlock_4Ucon_1x04_P3.50mm_Horizontal, F.Cu at (121.0, 170.0)
- added J5: MOT1, TerminalBlock_4Ucon:TerminalBlock_4Ucon_1x04_P3.50mm_Horizontal, F.Cu at (104.2, 179.0)
- added J6: MOT2, TerminalBlock_4Ucon:TerminalBlock_4Ucon_1x04_P3.50mm_Horizontal, F.Cu at (157.9, 155.7)
- added J7: MOT3, TerminalBlock_4Ucon:TerminalBlock_4Ucon_1x04_P3.50mm_Horizontal, F.Cu at (121.0, 179.0)
- added J8: MO0_SW_FW, Connector_Molex:Molex_Nano-Fit_105309-xx03_1x03_P2.50mm_Vertical, F.Cu at (140.2, 168.3)
- added J9: MO1_SW_FW, Connector_Molex:Molex_Nano-Fit_105309-xx03_1x03_P2.50mm_Vertical, F.Cu at (177.1, 145.0)
- added JP1: NC, Jumper:SolderJumper-2_P1.3mm_Bridged_RoundedPad1.0x1.5mm, F.Cu at (132.1, 195.6)
- added JP2: NC, Jumper:SolderJumper-2_P1.3mm_Bridged_RoundedPad1.0x1.5mm, F.Cu at (136.4, 195.6)
- added JP3: NC, Jumper:SolderJumper-2_P1.3mm_Bridged_RoundedPad1.0x1.5mm, F.Cu at (140.8, 195.6)
- added JP4: NC, Jumper:SolderJumper-2_P1.3mm_Bridged_RoundedPad1.0x1.5mm, F.Cu at (145.1, 195.6)
- added Q1: BSS138, Package_TO_SOT_SMD:SOT-23, F.Cu at (197.4, 147.5)
- added R1: R_10K, Resistor_SMD:R_0805_2012Metric_Pad1.20x1.40mm_HandSolder, F.Cu at (192.8, 143.7)
- added R2: R_10K, Resistor_SMD:R_0805_2012Metric_Pad1.20x1.40mm_HandSolder, F.Cu at (192.8, 146.7)
- added R3: R_10K, Resistor_SMD:R_0805_2012Metric_Pad1.20x1.40mm_HandSolder, F.Cu at (197.6, 143.7)
Connections:
- net /0(Rx0) renamed /Arduino Shield Connections/0(Rx0)
- net /1(Tx0) renamed /Arduino Shield Connections/1(Tx0)
- net /12(**) renamed /Arduino Shield Connections/12(**)
- net /13(**) renamed /Arduino Shield Connections/13(**)
- net /14(Tx3) renamed /Arduino Shield Connections/14(Tx3)
- net /15(Rx3) renamed /Arduino Shield Connections/15(Rx3)
- net /16(Tx2) renamed /Arduino Shield Connections/16(Tx2)
- net /17(Rx2) renamed /Arduino Shield Connections/17(Rx2)
- net /18(Tx1) renamed /Arduino Shield Connections/18(Tx1)
- net /19(Rx1) renamed /Arduino Shield Connections/19(Rx1)
- net /20(SDA) renamed /Arduino Shield Connections/20(SDA)
- net /21(SCL) renamed /Arduino Shield Connections/21(SCL)
- net /46 renamed /Arduino Shield Connections/46
- net /47 renamed /Arduino Shield Connections/47
- net /48 renamed /Arduino Shield Connections/48
- net /49 renamed /Arduino Shield Connections/49
- net /50(MISO) renamed /Arduino Shield Connections/50(MISO)
- net /51(MOSI) renamed /Arduino Shield Connections/51(MOSI)
- net /52(SCK) renamed /Arduino Shield Connections/52(SCK)
- net /53(SS) renamed /Arduino Shield Connections/53(SS)
- net /A0 renamed /Arduino Shield Connections/A0
- net /A1 renamed /Arduino Shield Connections/A1
- net /A10 renamed /Arduino Shield Connections/A10
- net /A11 renamed /Arduino Shield Connections/A11
- net /A12 renamed /Arduino Shield Connections/A12
- net /A13 renamed /Arduino Shield Connections/A13
- net /A14 renamed /Arduino Shield Connections/A14
- net /A15 renamed /Arduino Shield Connections/A15
- net /A2 renamed /Arduino Shield Connections/A2
- net /A3 renamed /Arduino Shield Connections/A3
- net /A4 renamed /Arduino Shield Connections/A4
- net /A5 renamed /Arduino Shield Connections/A5
- net /A6 renamed /Arduino Shield Connections/A6
- net /A7 renamed /Arduino Shield Connections/A7
- net /A8 renamed /Arduino Shield Connections/A8
- net /A9 renamed /Arduino Shield Connections/A9
- net /AREF renamed /Arduino Shield Connections/AREF
- net /IOREF renamed /Arduino Shield Connections/IOREF
- net /Reset renamed /Arduino Shield Connections/Reset
- net /SCL renamed /Arduino Shield Connections/SCL
- net /SDA renamed /Arduino Shield Connections/SDA
- net /Vin renamed /Arduino Shield Connections/Vin
- net GND renamed PWR_SW_L
- P1 pad 11: /44 -> MOT1_MS3
- P1 pad 12: /45 -> ~MOT3_EN
- P1 pad 13: /42 -> MOT1_MS2
- P1 pad 14: /43 -> MOT3_STEP
- P1 pad 15: /40 -> MOT1_MS1
- P1 pad 16: /41 -> MOT3_DIR
- P1 pad 17: /38 -> MOT1_DIR
- P1 pad 18: /39 -> MOT3_MS1
- P1 pad 19: /36 -> MOT1_STEP
- P1 pad 20: /37 -> MOT3_MS2
- P1 pad 21: /34 -> ~MOT1_EN
- P1 pad 22: /35 -> MOT3_MS3
- P1 pad 23: /32 -> MOT0_MS3
- P1 pad 24: /33 -> ~MOT2_EN
- P1 pad 25: /30 -> MOT0_MS2
- P1 pad 26: /31 -> MOT2_STEP
- P1 pad 27: /28 -> MOT0_MS1
- P1 pad 28: /29 -> MOT2_DIR
- P1 pad 29: /26 -> MOT0_DIR
- P1 pad 30: /27 -> MOT2_MS1
- P1 pad 31: /24 -> MOT0_STEP
- P1 pad 32: /25 -> MOT2_MS2
- P1 pad 33: /22 -> ~MOT0_EN
- P1 pad 34: /23 -> MOT2_MS3
- P5 pad 10: /8(**) -> MOT3_SWITCH_FW
- P5 pad 7: /11(**) -> ESTOP_L
- P5 pad 8: /10(**) -> PWR_SW
- P5 pad 9: /9(**) -> MOT3_SWITCH_BW
- P6 pad 1: /7(**) -> MOT2_SWITCH_BW
- P6 pad 2: /6(**) -> MOT2_SWITCH_FW
- P6 pad 3: /5(**) -> MOT1_SWITCH_BW
- P6 pad 4: /4(**) -> MOT1_SWITCH_FW
- P6 pad 5: /3(**) -> MOT0_SWITCH_BW
- P6 pad 6: /2(**) -> MOT0_SWITCH_FW
Routing:
- added copper zone on B.Cu, net PWR_SW_L
