File: hardware/control_board/control_board.sch (KiCad schematic (older format))
At the start: 13 parts, among them P1 Digital, P10 CONN_01X01, P11 CONN_01X01, P12 CONN_01X01, P13 CONN_01X01, P2 Power, P3 Analog, P4 Analog, P5 PWM, P6 PWM, P7 Communication, P8 CONN_01X01, P9 CONN_01X01

Commit message: control board schematic
Parts:
- removed P1: Digital, Socket_Arduino_Mega:Socket_Strip_Arduino_2x18, symbol Connector_Generic:Conn_02x18_Odd_Even
- removed P10, P11, P12, P13, P8, P9: CONN_01X01, Socket_Arduino_Mega:Arduino_1pin, symbol Connector_Generic:Conn_01x01
- removed P2: Power, Socket_Arduino_Mega:Socket_Strip_Arduino_1x08, symbol Connector_Generic:Conn_01x08
- removed P3, P4: Analog, Socket_Arduino_Mega:Socket_Strip_Arduino_1x08, symbol Connector_Generic:Conn_01x08
- removed P5: PWM, Socket_Arduino_Mega:Socket_Strip_Arduino_1x10, symbol Connector_Generic:Conn_01x10
- removed P6: PWM, Socket_Arduino_Mega:Socket_Strip_Arduino_1x08, symbol Connector_Generic:Conn_01x08
- removed P7: Communication, Socket_Arduino_Mega:Socket_Strip_Arduino_1x08, symbol Connector_Generic:Conn_01x08
Connections:
- no-connect marks 7 -> 0
Other:
- note removed: "1"
- note removed: "Holes"
- note removed: "Shield for Arduino Mega Rev 3"
