File: hardware/control_board/drivers.sch (KiCad schematic (older format))
At the start: 12 parts

Commit message: add ps on led
Parts:
- removed C1, C2, C3: 100uF, Capacitor_THT:CP_Radial_D12.5mm_P5.00mm, symbol Device:CP1_Small
- renumbered C4 to C1
Connections:
- wire segments 48 -> 34
Changed lines of the file:
@@
 	1    0    0    -1
 $EndComp
-Wire Wire Line
-	2500 2600 2500 2750
 $Comp
 L power:GND #PWR02
@@
 $EndComp
 Wire Wire Line
-	2650 2750 2500 2750
-Connection ~ 2500 2750
-Wire Wire Line
-	2500 2750 2500 2900
-$Comp
-L power:GND #PWR05
-U 1 1 61929737
-P 3000 2900
-F 0 "#PWR05" H 3000 2650 50  0001 C CNN
-F 1 "GND" H 3005 2727 50  0000 C CNN
-F 2 "" H 3000 2900 50  0001 C CNN
-F 3 "" H 3000 2900 50  0001 C CNN
-	1    3000 2900
-	1    0    0    -1
-$EndComp
-Wire Wire Line
-	3000 2900 3000 2750
-Wire Wire Line
-	3000 2750 2850 2750
-Wire Wire Line
 	2500 4400 2500 4550
 $Comp
@@
 	1    0    0    -1
 $EndComp
-Wire Wire Line
-	4500 2600 4500 2750
 $Comp
 L power:GND #PWR07
@@
 $EndComp
 Wire Wire Line
-	4650 2750 4500 2750
-Connection ~ 4500 2750
-Wire Wire Line
-	4500 2750 4500 2900
-$Comp
-L power:GND #PWR010
-U 1 1 6193D6DB
-P 5000 2900
-F 0 "#PWR010" H 5000 2650 50  0001 C CNN
-F 1 "GND" H 5005 2727 50  0000 C CNN
-F 2 "" H 5000 2900 50  0001 C CNN
-F 3 "" H 5000 2900 50  0001 C CNN
-	1    5000 2900
-	1    0    0    -1
-$EndComp
-Wire Wire Line
-	5000 2900 5000 2750
-Wire Wire Line
-	5000 2750 4850 2750
-Wire Wire Line
 	4500 4400 4500 4550
 $Comp
@@
 	1    0    0    -1
 $EndComp
-Wire Wire Line
-	6500 2600 6500 2750
 $Comp
 L power:GND #PWR012
@@
 $EndComp
 Wire Wire Line
-	6650 2750 6500 2750
-Connection ~ 6500 2750
-Wire Wire Line
-	6500 2750 6500 2900
-$Comp
-L power:GND #PWR015
-U 1 1 619448A4
-P 7000 2900
-F 0 "#PWR015" H 7000 2650 50  0001 C CNN
-F 1 "GND" H 7005 2727 50  0000 C CNN
-F 2 "" H 7000 2900 50  0001 C CNN
-F 3 "" H 7000 2900 50  0001 C CNN
-	1    7000 2900
-	1    0    0    -1
-$EndComp
-Wire Wire Line
-	7000 2900 7000 2750
-Wire Wire Line
-	7000 2750 6850 2750
-Wire Wire Line
 	6500 4400 6500 4550
 $Comp
@@
 	1    0    0    -1
 $EndComp
-Wire Wire Line
-	8500 2600 8500 2750
 $Comp
 L power:GND #PWR017
@@
 	1    0    0    -1
 $EndComp
-Wire Wire Line
-	8650 2750 8500 2750
-Connection ~ 8500 2750
-Wire Wire Line
-	8500 2750 8500 2900
-$Comp
-L power:GND #PWR020
-U 1 1 6194E65E
-P 9000 2900
-F 0 "#PWR020" H 9000 2650 50  0001 C CNN
-F 1 "GND" H 9005 2727 50  0000 C CNN
-F 2 "" H 9000 2900 50  0001 C CNN
-F 3 "" H 9000 2900 50  0001 C CNN
-	1    9000 2900
-	1    0    0    -1
-$EndComp
-Wire Wire Line
-	9000 2900 9000 2750
-Wire Wire Line
-	9000 2750 8850 2750
 Wire Wire Line
 	8500 4400 8500 4550
@@
 Wire Wire Line
 	7550 3300 7900 3300
+Wire Wire Line
+	2500 2600 2500 2900
+Wire Wire Line
+	4500 2600 4500 2900
+Wire Wire Line
+	6500 2600 6500 2900
+$Comp
+L power:GND #PWR020
+U 1 1 6194E65E
+P 9600 2850
+F 0 "#PWR020" H 9600 2600 50  0001 C CNN
+F 1 "GND" H 9605 2677 50  0000 C CNN
+F 2 "" H 9600 2850 50  0001 C CNN
+F 3 "" H 9600 2850 50  0001 C CNN
+	1    9600 2850
+	1    0    0    -1
+$EndComp
+Wire Wire Line
+	9600 2550 9600 2450
 $Comp
 L Device:CP1_Small C1
-U 1 1 61AB75C2
-P 2750 2750
-F 0 "C1" V 2850 2750 50  0000 C CNN
-F 1 "100uF" V 2650 2750 50  0000 C CNN
-F 2 "Capacitor_THT:CP_Radial_D12.5mm_P5.00mm" H 2750 2750 50  0001 C CNN
-F 3 "~" H 2750 2750 50  0001 C CNN
-	1    2750 2750
-	0    -1   -1   0
-$EndComp
-$Comp
-L Device:CP1_Small C2
-U 1 1 61AB9BEA
-P 4750 2750
-F 0 "C2" V 4850 2750 50  0000 C CNN
-F 1 "100uF" V 4650 2750 50  0000 C CNN
-F 2 "Capacitor_THT:CP_Radial_D12.5mm_P5.00mm" H 4750 2750 50  0001 C CNN
-F 3 "~" H 4750 2750 50  0001 C CNN
-	1    4750 2750
-	0    -1   -1   0
-$EndComp
-$Comp
-L Device:CP1_Small C3
-U 1 1 61ABA585
-P 6750 2750
-F 0 "C3" V 6850 2750 50  0000 C CNN
-F 1 "100uF" V 6650 2750 50  0000 C CNN
-F 2 "Capacitor_THT:CP_Radial_D12.5mm_P5.00mm" H 6750 2750 50  0001 C CNN
-F 3 "~" H 6750 2750 50  0001 C CNN
-	1    6750 2750
-	0    -1   -1   0
-$EndComp
-$Comp
-L Device:CP1_Small C4
 U 1 1 61ABB008
-P 8750 2750
-F 0 "C4" V 8850 2750 50  0000 C CNN
-F 1 "100uF" V 8650 2750 50  0000 C CNN
-F 2 "Capacitor_THT:CP_Radial_D12.5mm_P5.00mm" H 8750 2750 50  0001 C CNN
-F 3 "~" H 8750 2750 50  0001 C CNN
-	1    8750 2750
-	0    -1   -1   0
+P 9600 2650
+F 0 "C1" V 9700 2650 50  0000 C CNN
+F 1 "100uF" V 9500 2650 50  0000 C CNN
+F 2 "Capacitor_THT:CP_Radial_D12.5mm_P5.00mm" H 9600 2650 50  0001 C CNN
+F 3 "~" H 9600 2650 50  0001 C CNN
+	1    9600 2650
+	1    0    0    -1
+$EndComp
+Wire Wire Line
+	9600 2750 9600 2850
+Wire Wire Line
+	8500 2600 8500 2900
+$Comp
+L power:+12V #PWR?
+U 1 1 6188338D
+P 9600 2450
+F 0 "#PWR?" H 9600 2300 50  0001 C CNN
+F 1 "+12V" H 9615 2623 50  0000 C CNN
+F 2 "" H 9600 2450 50  0001 C CNN
+F 3 "" H 9600 2450 50  0001 C CNN
+	1    9600 2450
+	1    0    0    -1
 $EndComp
 $EndSCHEMATC

Commit message: finish layout, add fusing
Parts:
- added R5, R6, R7, R8: R_10K, Resistor_SMD:R_0805_2012Metric_Pad1.20x1.40mm_HandSolder, symbol Device:R_Small_US
Connections:
- wire segments 34 -> 46
Changed lines of the file:
@@
 	1    0    0    -1
 $EndComp
+$Comp
+L Device:R_Small_US R5
+U 1 1 619F4ED4
+P 1550 2450
+F 0 "R5" H 1618 2496 50  0000 L CNN
+F 1 "R_10K" H 1618 2405 50  0000 L CNN
+F 2 "Resistor_SMD:R_0805_2012Metric_Pad1.20x1.40mm_HandSolder" H 1550 2450 50  0001 C CNN
+F 3 "~" H 1550 2450 50  0001 C CNN
+	1    1550 2450
+	1    0    0    -1
+$EndComp
+Text GLabel 1600 2700 2    40   Input ~ 0
+~MOT0_EN
+Wire Wire Line
+	1600 2700 1550 2700
+Wire Wire Line
+	1550 2700 1550 2550
+$Comp
+L power:+5V #PWR053
+U 1 1 619F6B47
+P 1550 2250
+F 0 "#PWR053" H 1550 2100 50  0001 C CNN
+F 1 "+5V" H 1565 2423 50  0000 C CNN
+F 2 "" H 1550 2250 50  0001 C CNN
+F 3 "" H 1550 2250 50  0001 C CNN
+	1    1550 2250
+	1    0    0    -1
+$EndComp
+Wire Wire Line
+	1550 2250 1550 2350
+$Comp
+L Device:R_Small_US R6
+U 1 1 61A03D1C
+P 3550 2450
+F 0 "R6" H 3618 2496 50  0000 L CNN
+F 1 "R_10K" H 3618 2405 50  0000 L CNN
+F 2 "Resistor_SMD:R_0805_2012Metric_Pad1.20x1.40mm_HandSolder" H 3550 2450 50  0001 C CNN
+F 3 "~" H 3550 2450 50  0001 C CNN
+	1    3550 2450
+	1    0    0    -1
+$EndComp
+Text GLabel 3600 2700 2    40   Input ~ 0
+~MOT1_EN
+Wire Wire Line
+	3600 2700 3550 2700
+Wire Wire Line
+	3550 2700 3550 2550
+$Comp
+L power:+5V #PWR054
+U 1 1 61A03D25
+P 3550 2250
+F 0 "#PWR054" H 3550 2100 50  0001 C CNN
+F 1 "+5V" H 3565 2423 50  0000 C CNN
+F 2 "" H 3550 2250 50  0001 C CNN
+F 3 "" H 3550 2250 50  0001 C CNN
+	1    3550 2250
+	1    0    0    -1
+$EndComp
+Wire Wire Line
+	3550 2250 3550 2350
+$Comp
+L Device:R_Small_US R7
+U 1 1 61A06B71
+P 5550 2450
+F 0 "R7" H 5618 2496 50  0000 L CNN
+F 1 "R_10K" H 5618 2405 50  0000 L CNN
+F 2 "Resistor_SMD:R_0805_2012Metric_Pad1.20x1.40mm_HandSolder" H 5550 2450 50  0001 C CNN
+F 3 "~" H 5550 2450 50  0001 C CNN
+	1    5550 2450
+	1    0    0    -1
+$EndComp
+Text GLabel 5600 2700 2    40   Input ~ 0
+~MOT2_EN
+Wire Wire Line
+	5600 2700 5550 2700
+Wire Wire Line
+	5550 2700 5550 2550
+$Comp
+L power:+5V #PWR055
+U 1 1 61A06B7A
+P 5550 2250
+F 0 "#PWR055" H 5550 2100 50  0001 C CNN
+F 1 "+5V" H 5565 2423 50  0000 C CNN
+F 2 "" H 5550 2250 50  0001 C CNN
+F 3 "" H 5550 2250 50  0001 C CNN
+	1    5550 2250
+	1    0    0    -1
+$EndComp
+Wire Wire Line
+	5550 2250 5550 2350
+$Comp
+L Device:R_Small_US R8
+U 1 1 61A096B9
+P 7550 2450
+F 0 "R8" H 7618 2496 50  0000 L CNN
+F 1 "R_10K" H 7618 2405 50  0000 L CNN
+F 2 "Resistor_SMD:R_0805_2012Metric_Pad1.20x1.40mm_HandSolder" H 7550 2450 50  0001 C CNN
+F 3 "~" H 7550 2450 50  0001 C CNN
+	1    7550 2450
+	1    0    0    -1
+$EndComp
+Text GLabel 7600 2700 2    40   Input ~ 0
+~MOT3_EN
+Wire Wire Line
+	7600 2700 7550 2700
+Wire Wire Line
+	7550 2700 7550 2550
+$Comp
+L power:+5V #PWR056
+U 1 1 61A096C2
+P 7550 2250
+F 0 "#PWR056" H 7550 2100 50  0001 C CNN
+F 1 "+5V" H 7565 2423 50  0000 C CNN
+F 2 "" H 7550 2250 50  0001 C CNN
+F 3 "" H 7550 2250 50  0001 C CNN
+	1    7550 2250
+	1    0    0    -1
+$EndComp
+Wire Wire Line
+	7550 2250 7550 2350
 $EndSCHEMATC
